File: KiCad/RIAAPre.sch (KiCad schematic (older format))
At the start: 42 parts, among them K1 RCA, K2 RCA, K3 16VAC, U1 NJM4580, U2 MC7815, U3 MC7915

Commit message: Directory cleanup and ignore additions.
Parts:
- U1: symbol LM358 -> LM358-RESCUE-RIAAPre
Changed lines of the file:
@@
 $EndComp
 $Comp
-L LM358 U1
+L LM358-RESCUE-RIAAPre U1
 U 2 1 54A3A559
 P 3650 4750
@@
 $EndComp
 $Comp
-L LM358 U1
+L LM358-RESCUE-RIAAPre U1
 U 1 1 54AB34DA
 P 3600 1300
